Commit message: error calculation function

File: kuka-bartender/bartender_description/robot/bartender.urdf.xacro (robot description, xacro)
@@ -36,22 +36,22 @@
   <!-- BOTTLES -->
   <xacro:model_bottle name="vodka" parent="bartender_anchor">
-    <origin xyz="-1.15 0.15 0.22" rpy="0 0 0"/>
+    <origin xyz="-1.0 0.15 0.22" rpy="0 0 0"/>
     <material name="Vito/LightGrey"/>
   </xacro:model_bottle>
   <xacro:model_bottle name="lemon" parent="bartender_anchor">
-    <origin xyz="-1.15 -0.15 0.22" rpy="0 0 0"/>
+    <origin xyz="-1.0 -0.15 0.22" rpy="0 0 0"/>
     <material name="Vito/Orange"/>
   </xacro:model_bottle>
   <xacro:model_bottle name="rum" parent="bartender_anchor">
-    <origin xyz="-1.15 0.3 0.22" rpy="0 0 0"/>
+    <origin xyz="-1.0 0.3 0.22" rpy="0 0 0"/>
     <material name="Vito/Green"/>
   </xacro:model_bottle>
   <xacro:model_bottle name="coca" parent="bartender_anchor">
-    <origin xyz="-1.15 -0.3 0.22" rpy="0 0 0"/>
+    <origin xyz="-1.0 -0.3 0.22" rpy="0 0 0"/>
     <material name="Vito/Yellow"/>
   </xacro:model_bottle>
   <!-- GLASS -->
   <xacro:model_glass name="glass" parent="bartender_anchor">
-    <origin xyz="-1.05 0 0.15" rpy="0 0 0"/>
+    <origin xyz="-0.9 0 0.15" rpy="0 0 0"/>
   </xacro:model_glass>
   <!-- TORSO -->

Commit message: modified EE for chain controller and added new cfg_parameter

File: kuka-bartender/bartender_description/robot/bartender.urdf.xacro (robot description, xacro)
@@ -36,17 +36,17 @@
   <!-- BOTTLES -->
   <xacro:model_bottle name="vodka" parent="bartender_anchor">
-    <origin xyz="-1.0 0.15 0.22" rpy="0 0 0"/>
+    <origin xyz="-1 0.15 0.22" rpy="0 0 0"/>
     <material name="Vito/LightGrey"/>
   </xacro:model_bottle>
   <xacro:model_bottle name="lemon" parent="bartender_anchor">
-    <origin xyz="-1.0 -0.15 0.22" rpy="0 0 0"/>
+    <origin xyz="-1 -0.15 0.22" rpy="0 0 0"/>
     <material name="Vito/Orange"/>
   </xacro:model_bottle>
   <xacro:model_bottle name="rum" parent="bartender_anchor">
-    <origin xyz="-1.0 0.3 0.22" rpy="0 0 0"/>
+    <origin xyz="-1 0.3 0.22" rpy="0 0 0"/>
     <material name="Vito/Green"/>
   </xacro:model_bottle>
   <xacro:model_bottle name="coca" parent="bartender_anchor">
-    <origin xyz="-1.0 -0.3 0.22" rpy="0 0 0"/>
+    <origin xyz="-1 -0.3 0.22" rpy="0 0 0"/>
     <material name="Vito/Yellow"/>
   </xacro:model_bottle>

Commit message: grasping poses added. FIXME first action bugged

File: kuka-bartender/bartender_description/robot/bartender.urdf.xacro (robot description, xacro)
@@ -34,25 +34,4 @@
   <origin xyz="-1.25 0.55 0.07" rpy="0 0 0"/>
   </xacro:model_table>
-  <!-- BOTTLES -->
-  <xacro:model_bottle name="vodka" parent="bartender_anchor">
-    <origin xyz="-1 0.15 0.22" rpy="0 0 0"/>
-    <material name="Vito/LightGrey"/>
-  </xacro:model_bottle>
-  <xacro:model_bottle name="lemon" parent="bartender_anchor">
-    <origin xyz="-1 -0.15 0.22" rpy="0 0 0"/>
-    <material name="Vito/Orange"/>
-  </xacro:model_bottle>
-  <xacro:model_bottle name="rum" parent="bartender_anchor">
-    <origin xyz="-1 0.3 0.22" rpy="0 0 0"/>
-    <material name="Vito/Green"/>
-  </xacro:model_bottle>
-  <xacro:model_bottle name="coca" parent="bartender_anchor">
-    <origin xyz="-1 -0.3 0.22" rpy="0 0 0"/>
-    <material name="Vito/Yellow"/>
-  </xacro:model_bottle>
-  <!-- GLASS -->
-  <xacro:model_glass name="glass" parent="bartender_anchor">
-    <origin xyz="-0.9 0 0.15" rpy="0 0 0"/>
-  </xacro:model_glass>
   <!-- TORSO -->
   <xacro:model_torso name="torso" parent="bartender_anchor">

Commit message: services and new functions (stable version)

File: kuka-bartender/bartender_description/robot/bartender.urdf.xacro (robot description, xacro)
@@ -45,5 +45,5 @@
   <!-- LEFT SOFTHAND -->
   <xacro:soft_hand parent="left_arm_7_link" name="left_hand" left="true" withAdaptiveTransmission="true" useMimicTag="$(arg use_mimic_tag)">
-    <origin xyz="0 0 0" rpy="0 0 0"/>
+    <origin xyz="0 0 0" rpy="0 0 -3.14"/>
   </xacro:soft_hand>
   <!-- RIGHT ARM -->
